File: stabielator_v1_pcb/stabielator/haptic.kicad_sch (KiCad schematic)
At the start: 33 parts, among them J3 Motor 1, J4 Motor 2, J5 Motor 3, J6 Motor 4, U1 DRV2605LDGS, U4 TCA9546APW, U5 DRV2605LDGS, U6 DRV2605LDGS, U7 DRV2605LDGS

Commit message: Finished for review
Connections:
- net +3.3V: now also R50.1, R51.1, R52.1, R53.1, R54.1, R55.1, R56.1, R57.1
- net VCC: no longer R50.1, R51.1, R52.1, R53.1, R54.1, R55.1, R56.1, R57.1, U1.5 (EN), U5.5 (EN), U6.5 (EN), U7.5 (EN)
- new net POWERSTATE: U1.5 (EN), U5.5 (EN), U6.5 (EN), U7.5 (EN)
Other:
- note added: "Verplaatst van batt naar 3.3v om standby instabiliteit te voorkomen"
