File: stabielator_v1_pcb/stabielator/power.kicad_sch (KiCad schematic)
At the start: 46 parts, among them J1 USB_C_Receptacle_USB2.0_16P, J2 Battery, Q1 2N7002, Q2 2N7002, SW1 PWR, U10 BQ24074RGT, U11 TPS22917DBV, U13 TLV62569DBV, U8 USBLC6-2SC6, U9 TPS3424A11C13ADRLR

Commit message: Finished for review
Parts:
- removed C43: 1nF, Capacitor_SMD:C_0603_1608Metric, symbol Device:C
- removed U11: TPS22917DBV, Package_TO_SOT_SMD:SOT-23-6, symbol Power_Management:TPS22917DBV
- added R26, R27: 22R, Resistor_SMD:R_0603_1608Metric, symbol Device:R
Connections:
- net BATT_VCC is gone; now on net VCC: C39.2, C41.1, C44.2, D5.2 (A), R78.1, R79.1, U10.10 (OUT), U10.11 (OUT), U9.3 (VDD)
- net USB_D+: now also R27.1; no longer U8.4 (I/O2)
- net USB_D-: now also R26.2; no longer U8.6 (I/O1)
- net VCC: no longer U13.1 (EN)
- net POWERSTATE: now reaches U9.6 (RST)
- net POWERSTATE: now also U13.1 (EN)
- new net: R27.2, U8.4 (I/O2)
- new net: R26.1, U8.6 (I/O1)
Other:
- note added: "ON/OFF Controller"
- note removed: "Load switch"
- moved on the sheet: C38, C41, C44, C45, Q2, R76, R77, R78, SW1, U9
