File: PCB/power.kicad_sch (KiCad schematic)
At the start: 46 parts, among them J1 S2B-PH, J5 USB4105-GF-A, Q1 2N7002, SW2 PWR, U10 USBLC6-2SC6, U3 BQ24074RGT, U4 TPS63001, U9 TPS3424A11C13ADRLR

Commit message: Geographical reannotation
Parts:
- renumbered C14 to C15, C27 to C26, C28 to C30, C7 to C5, D3 to D2, R19 to R15, R21 to R16, R17 to R18, R28 to R20, R24 to R21, R15 to R22, R26 to R24, R31 to R25, R32 to R26, R16 to R27, R30 to R32, R4 to R6, R5 to R7, R10 to R9, TP12 to TP1, TP3 to TP10, TP13 to TP11, TP11 to TP12, TP16 to TP13, TP17 to TP2, TP15 to TP7, TP14 to TP9, U9 to U11, U10 to U9
Changed lines of the file:
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@@
 	(title_block
 		(title "${Project_name}")
-		(date "2026-09-07")
+		(date "2026-09-20")
 		(rev "${Project_revision}")
 		(company "${Company_name}")
@@
 		(in_pos_files yes)
 		(dnp no)
-		(property "Reference" "R21"
+		(property "Reference" "R16"
 			(at 54.61 60.96 0)
 			(show_name no)
@@
 			(project "stabielator"
 				(path "/c0e871b7-8ed4-4f9b-ae4f-e503a34d56f3/73929003-3baa-4f9c-89cc-74ae5f550b44"
-					(reference "R21")
+					(reference "R16")
 					(unit 1)
 				)
@@
 		(in_pos_files yes)
 		(dnp no)
-		(property "Reference" "TP12"
+		(property "Reference" "TP1"
 			(at 248.666 104.902 0)
 			(show_name no)
@@
 			(project "stabielator"
 				(path "/c0e871b7-8ed4-4f9b-ae4f-e503a34d56f3/73929003-3baa-4f9c-89cc-74ae5f550b44"
-					(reference "TP12")
+					(reference "TP1")
 					(unit 1)
 				)
@@
 		(in_pos_files yes)
 		(dnp no)
-		(property "Reference" "C7"
+		(property "Reference" "C5"
 			(at 265.811 123.2916 0)
 			(show_name no)
@@
 			(project "stabielator"
 				(path "/c0e871b7-8ed4-4f9b-ae4f-e503a34d56f3/73929003-3baa-4f9c-89cc-74ae5f550b44"
-					(reference "C7")
+					(reference "C5")
 					(unit 1)
 				)
@@
 		(in_pos_files yes)
 		(dnp no)
-		(property "Reference" "C27"
+		(property "Reference" "C26"
 			(at 245.11 44.45 90)
 			(show_name no)
@@
 			(project "stabielator"
 				(path "/c0e871b7-8ed4-4f9b-ae4f-e503a34d56f3/73929003-3baa-4f9c-89cc-74ae5f550b44"
-					(reference "C27")
+					(reference "C26")
 					(unit 1)
 				)
@@
 		(in_pos_files yes)
 		(dnp no)
-		(property "Reference" "R16"
+		(property "Reference" "R27"
 			(at 107.95 118.11 90)
 			(show_name no)
@@
 			(project "stabielator"
 				(path "/c0e871b7-8ed4-4f9b-ae4f-e503a34d56f3/73929003-3baa-4f9c-89cc-74ae5f550b44"
-					(reference "R16")
+					(reference "R27")
 					(unit 1)
 				)
@@
 		(in_pos_files yes)
 		(dnp no)
-		(property "Reference" "TP15"
+		(property "Reference" "TP7"
 			(at 169.926 40.386 90)
 			(show_name no)
@@
 			(project "stabielator"
 				(path "/c0e871b7-8ed4-4f9b-ae4f-e503a34d56f3/73929003-3baa-4f9c-89cc-74ae5f550b44"
-					(reference "TP15")
+					(reference "TP7")
 					(unit 1)
 				)
@@
 		(in_pos_files yes)
 		(dnp no)
-		(property "Reference" "R31"
+		(property "Reference" "R25"
 			(at 181.61 55.88 0)
 			(show_name no)
@@
 			(project "stabielator"
 				(path "/c0e871b7-8ed4-4f9b-ae4f-e503a34d56f3/73929003-3baa-4f9c-89cc-74ae5f550b44"
-					(reference "R31")
+					(reference "R25")
 					(unit 1)
 				)
@@
 		(in_pos_files yes)
 		(dnp no)
-		(property "Reference" "TP14"
+		(property "Reference" "TP9"
 			(at 204.724 47.752 90)
 			(show_name no)
@@
 			(project "stabielator"
 				(path "/c0e871b7-8ed4-4f9b-ae4f-e503a34d56f3/73929003-3baa-4f9c-89cc-74ae5f550b44"
-					(reference "TP14")
+					(reference "TP9")
 					(unit 1)
 				)
@@
 		(in_pos_files yes)
 		(dnp no)
-		(property "Reference" "R5"
+		(property "Reference" "R7"
 			(at 140.97 63.5 0)
 			(show_name no)
@@
 			(project "stabielator"
 				(path "/c0e871b7-8ed4-4f9b-ae4f-e503a34d56f3/73929003-3baa-4f9c-89cc-74ae5f550b44"
-					(reference "R5")
+					(reference "R7")
 					(unit 1)
 				)
@@
 		(in_pos_files yes)
 		(dnp no)
-		(property "Reference" "C28"
+		(property "Reference" "C30"
 			(at 269.24 53.848 0)
 			(show_name no)
@@
 			(project "stabielator"
 				(path "/c0e871b7-8ed4-4f9b-ae4f-e503a34d56f3/73929003-3baa-4f9c-89cc-74ae5f550b44"
-					(reference "C28")
+					(reference "C30")
 					(unit 1)
 				)
@@
 		(in_pos_files yes)
 		(dnp no)
-		(property "Reference" "R15"
+		(property "Reference" "R22"
 			(at 107.95 115.57 90)
 			(show_name no)
@@
 			(project "stabielator"
 				(path "/c0e871b7-8ed4-4f9b-ae4f-e503a34d56f3/73929003-3baa-4f9c-89cc-74ae5f550b44"
-					(reference "R15")
+					(reference "R22")
 					(unit 1)
 				)
@@
 		(dnp no)
 		(fields_autoplaced yes)
-		(property "Reference" "D3"
+		(property "Reference" "D2"
 			(at 143.51 75.2474 90)
 			(show_name no)
@@
 			(project "stabielator"
 				(path "/c0e871b7-8ed4-4f9b-ae4f-e503a34d56f3/73929003-3baa-4f9c-89cc-74ae5f550b44"
-					(reference "D3")
+					(reference "D2")
 					(unit 1)
 				)
@@
 		(in_pos_files yes)
 		(dnp no)
-		(property "Reference" "R19"
+		(property "Reference" "R15"
 			(at 102.87 55.88 0)
 			(show_name no)
@@
 			(project "stabielator"
 				(path "/c0e871b7-8ed4-4f9b-ae4f-e503a34d56f3/73929003-3baa-4f9c-89cc-74ae5f550b44"
-					(reference "R19")
+					(reference "R15")
 					(unit 1)
 				)
@@
 		(in_pos_files yes)
 		(dnp no)
-		(property "Reference" "U9"
+		(property "Reference" "U11"
 			(at 223.52 36.83 0)
 			(show_name no)
@@
 			(project "stabielator"
 				(path "/c0e871b7-8ed4-4f9b-ae4f-e503a34d56f3/73929003-3baa-4f9c-89cc-74ae5f550b44"
-					(reference "U9")
+					(reference "U11")
 					(unit 1)
 				)
@@
 		(dnp no)
 		(fields_autoplaced yes)
-		(property "Reference" "TP11"
+		(property "Reference" "TP12"
 			(at 115.57 106.9976 0)
 			(show_name no)
@@
 			(project "stabielator"
 				(path "/c0e871b7-8ed4-4f9b-ae4f-e503a34d56f3/73929003-3baa-4f9c-89cc-74ae5f550b44"
-					(reference "TP11")
+					(reference "TP12")
 					(unit 1)
 				)
@@
 		(in_pos_files yes)
 		(dnp no)
-		(property "Reference" "R30"
+		(property "Reference" "R32"
 			(at 194.31 35.56 0)
 			(show_name no)
@@
 			(project "stabielator"
 				(path "/c0e871b7-8ed4-4f9b-ae4f-e503a34d56f3/73929003-3baa-4f9c-89cc-74ae5f550b44"
-					(reference "R30")
+					(reference "R32")
 					(unit 1)
 				)
@@
 		(in_pos_files yes)
 		(dnp no)
-		(property "Reference" "R10"
+		(property "Reference" "R9"
 			(at 34.29 60.96 0)
 			(show_name no)
@@
 			(project "stabielator"
 				(path "/c0e871b7-8ed4-4f9b-ae4f-e503a34d56f3/73929003-3baa-4f9c-89cc-74ae5f550b44"
-					(reference "R10")
+					(reference "R9")
 					(unit 1)
 				)
@@
 		(dnp no)
 		(fields_autoplaced yes)
-		(property "Reference" "U10"
+		(property "Reference" "U9"
 			(at 95.6311 109.22 0)
 			(show_name no)
@@
 			(project "stabielator"
 				(path "/c0e871b7-8ed4-4f9b-ae4f-e503a34d56f3/73929003-3baa-4f9c-89cc-74ae5f550b44"
-					(reference "U10")
+					(reference "U9")
 					(unit 1)
 				)
@@
 		(in_pos_files yes)
 		(dnp no)
-		(property "Reference" "R24"
+		(property "Reference" "R21"
 			(at 95.25 139.7 0)
 			(show_name no)
@@
 			(project "stabielator"
 				(path "/c0e871b7-8ed4-4f9b-ae4f-e503a34d56f3/73929003-3baa-4f9c-89cc-74ae5f550b44"
-					(reference "R24")
+					(reference "R21")
 					(unit 1)
 				)
@@
 		(in_pos_files yes)
 		(dnp no)
-		(property "Reference" "TP16"
+		(property "Reference" "TP13"
 			(at 220.472 55.118 0)
 			(show_name no)
@@
 			(project "stabielator"
 				(path "/c0e871b7-8ed4-4f9b-ae4f-e503a34d56f3/73929003-3baa-4f9c-89cc-74ae5f550b44"
-					(reference "TP16")
+					(reference "TP13")
 					(unit 1)
 				)
@@
 		(in_pos_files yes)
 		(dnp no)
-		(property "Reference" "R26"
+		(property "Reference" "R24"
 			(at 41.91 137.16 0)
 			(show_name no)
@@
 			(project "stabielator"
 				(path "/c0e871b7-8ed4-4f9b-ae4f-e503a34d56f3/73929003-3baa-4f9c-89cc-74ae5f550b44"
-					(reference "R26")
+					(reference "R24")
 					(unit 1)
 				)
@@
 		(in_pos_files yes)
 		(dnp no)
-		(property "Reference" "R17"
+		(property "Reference" "R18"
 			(at 44.45 60.96 0)
 			(show_name no)
@@
 			(project "stabielator"
 				(path "/c0e871b7-8ed4-4f9b-ae4f-e503a34d56f3/73929003-3baa-4f9c-89cc-74ae5f550b44"
-					(reference "R17")
+					(reference "R18")
 					(unit 1)
 				)
@@
 		(in_pos_files yes)
 		(dnp no)
-		(property "Reference" "R4"
+		(property "Reference" "R6"
 			(at 199.39 118.11 0)
 			(show_name no)
@@
 			(project "stabielator"
 				(path "/c0e871b7-8ed4-4f9b-ae4f-e503a34d56f3/73929003-3baa-4f9c-89cc-74ae5f550b44"
-					(reference "R4")
+					(reference "R6")
 					(unit 1)
 				)
@@
 		(in_pos_files yes)
 		(dnp no)
-		(property "Reference" "TP3"
+		(property "Reference" "TP10"
 			(at 195.58 105.664 0)
 			(show_name no)
@@
 			(project "stabielator"
 				(path "/c0e871b7-8ed4-4f9b-ae4f-e503a34d56f3/73929003-3baa-4f9c-89cc-74ae5f550b44"
-					(reference "TP3")
+					(reference "TP10")
 					(unit 1)
 				)
@@
 		(in_pos_files yes)
 		(dnp no)
-		(property "Reference" "R28"
+		(property "Reference" "R20"
 			(at 87.63 139.7 0)
 			(show_name no)
@@
 			(project "stabielator"
 				(path "/c0e871b7-8ed4-4f9b-ae4f-e503a34d56f3/73929003-3baa-4f9c-89cc-74ae5f550b44"
-					(reference "R28")
+					(reference "R20")
 					(unit 1)
 				)
@@
 		(in_pos_files yes)
 		(dnp no)
-		(property "Reference" "TP17"
+		(property "Reference" "TP2"
 			(at 66.294 71.374 90)
 			(show_name no)
@@
 			(project "stabielator"
 				(path "/c0e871b7-8ed4-4f9b-ae4f-e503a34d56f3/73929003-3baa-4f9c-89cc-74ae5f550b44"
-					(reference "TP17")
+					(reference "TP2")
 					(unit 1)
 				)
@@
 		(in_pos_files yes)
 		(dnp no)
-		(property "Reference" "C14"
+		(property "Reference" "C15"
 			(at 188.341 123.2916 0)
 			(show_name no)
@@
 			(project "stabielator"
 				(path "/c0e871b7-8ed4-4f9b-ae4f-e503a34d56f3/73929003-3baa-4f9c-89cc-74ae5f550b44"
-					(reference "C14")
+					(reference "C15")
 					(unit 1)
 				)
@@
 		(in_pos_files yes)
 		(dnp no)
-		(property "Reference" "R32"
+		(property "Reference" "R26"
 			(at 171.45 45.72 90)
 			(show_name no)
@@
 			(project "stabielator"
 				(path "/c0e871b7-8ed4-4f9b-ae4f-e503a34d56f3/73929003-3baa-4f9c-89cc-74ae5f550b44"
-					(reference "R32")
+					(reference "R26")
 					(unit 1)
 				)
@@
 		(dnp no)
 		(fields_autoplaced yes)
-		(property "Reference" "TP13"
+		(property "Reference" "TP11"
 			(at 115.57 131.7624 0)
 			(show_name no)
@@
 			(project "stabielator"
 				(path "/c0e871b7-8ed4-4f9b-ae4f-e503a34d56f3/73929003-3baa-4f9c-89cc-74ae5f550b44"
-					(reference "TP13")
+					(reference "TP11")
 					(unit 1)
 				)

Commit message: Ready for production
Small readability and producability optimizations
Parts:
- C25: Manufacturer KEMET -> KEMET
- D2: Manifacturer Würth Elektronik -> (none); Manufacturer (none) -> Wurth
- J1: Manufacturer JST Sales America Inc. -> JST
- R1: value 100k 0.1% -> 100k; Digikey YAG1235CT-ND -> 311-100KHRCT-ND; Partnumber RT0603BRD07100KL -> RC0603FR-07100KL
- R2: value 300k 0.1% -> 300k; Digikey YAG1627CT-ND -> 311-300KHRTR-ND; Partnumber RT0603BRD07300KL -> RC0603FR-07300KL
- R20, R21: Digikey YAG3621CT-ND -> 311-5.10KHRTR-ND; Partnumber AC0603FR-075K1L -> RC0603FR-075K1L
- R22, R27: Digikey YAG3581CT-ND -> 311-22.0HRTR-ND; Partnumber AC0603FR-0722RL -> RC0603FR-0722RL
- U9: Digikey 5399-USBLC6-2SC6CT-ND -> 497-5235-2-ND; Manufacturer Shenzhen Slkormicro Semicon Co., Ltd. -> STMicroelectronics
Connections:
- net GND: now also SW2.MP
Other:
- note added: "Battery measurement"
- note removed: "Battery measurement (might need load switch or removal of feature)"
- moved on the sheet: C10, C11, C13, C15, C26, C30, C5, C8, C9, D2, J1, L1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
